Commit message: added inertia

File: dobot_viz/urdf/dobot_viz.urdf.xacro (robot description, xacro)
@@ -50,4 +50,10 @@
     <color rgba="0 1 0 1"/>
 </material>
+<link name="world"></link>
+<joint name="base_joint" type="fixed">
+    <origin xyz="0.0 0.0 0" rpy="0 0 0"/>
+    <parent link="world"/>
+    <child link="base_link"/>
+</joint>
 <link name="base_link">
     <visual>
@@ -57,4 +63,15 @@
         <material name="white"/>
     </visual>
+    <collision>
+            <origin xyz="0 0 0.05" rpy="0 0 0"/>
+            <geometry>
+                <box size="2.5 1.5 0.1" />
+            </geometry>
+        </collision>
+        <inertial>
+            <origin xyz="0 0 0.05" rpy="0 0 0"/>
+            <mass value="12" />
+            <inertia ixx="2.26" ixy="0.0" ixz="0.0" iyy="6.26" iyz="0.0" izz="8.5" />
+        </inertial>
 </link>
 <link name="front">
@@ -66,4 +83,15 @@
         <origin xyz="${by/2} 0 ${bh/2}"/>
     </visual>
+    <collision>
+            <origin xyz="0 0 0.05" rpy="0 0 0"/>
+            <geometry>
+                <box size="2.5 1.5 0.1" />
+            </geometry>
+        </collision>
+        <inertial>
+            <origin xyz="0 0 0.05" rpy="0 0 0"/>
+            <mass value="12" />
+            <inertia ixx="2.26" ixy="0.0" ixz="0.0" iyy="6.26" iyz="0.0" izz="8.5" />
+        </inertial>
 </link>
 <joint name="front_joint" type="fixed">
@@ -80,4 +108,15 @@
         <origin xyz="0 0 0"/>
     </visual>
+    <collision>
+            <origin xyz="0 0 0.05" rpy="0 0 0"/>
+            <geometry>
+                <box size="2.5 1.5 0.1" />
+            </geometry>
+        </collision>
+        <inertial>
+            <origin xyz="0 0 0.05" rpy="0 0 0"/>
+            <mass value="12" />
+            <inertia ixx="2.26" ixy="0.0" ixz="0.0" iyy="6.26" iyz="0.0" izz="8.5" />
+        </inertial>
 </link>
 <joint name="rotate_base__base" type="revolute">
@@ -96,4 +135,15 @@
         <origin xyz="0 ${-0.5*(wmw+rbr-0.5*wmw)} ${0.5*(rbh+wbh-bh-rbh+dmjr)}"/>
     </visual>
+    <collision>
+            <origin xyz="0 0 0.05" rpy="0 0 0"/>
+            <geometry>
+                <box size="2.5 1.5 0.1" />
+            </geometry>
+        </collision>
+        <inertial>
+            <origin xyz="0 0 0.05" rpy="0 0 0"/>
+            <mass value="12" />
+            <inertia ixx="2.26" ixy="0.0" ixz="0.0" iyy="6.26" iyz="0.0" izz="8.5" />
+        </inertial>
 </link>
 <link name="right_manipulator_handler">
@@ -105,4 +155,15 @@
         <origin xyz="0 ${0.5*(wmw+rbr-0.5*wmw)} ${0.5*(rbh+wbh-bh-rbh+dmjr)}"/>
     </visual>
+    <collision>
+            <origin xyz="0 0 0.05" rpy="0 0 0"/>
+            <geometry>
+                <box size="2.5 1.5 0.1" />
+            </geometry>
+        </collision>
+        <inertial>
+            <origin xyz="0 0 0.05" rpy="0 0 0"/>
+            <mass value="12" />
+            <inertia ixx="2.26" ixy="0.0" ixz="0.0" iyy="6.26" iyz="0.0" izz="8.5" />
+        </inertial>
 </link>
 <joint name="left_manipulator_handler__rotation_base" type="fixed">
@@ -124,4 +185,15 @@
         <origin rpy="1.57075 0 0" xyz="0 0 0"/>
     </visual>
+    <collision>
+            <origin xyz="0 0 0.05" rpy="0 0 0"/>
+            <geometry>
+                <box size="2.5 1.5 0.1" />
+            </geometry>
+        </collision>
+        <inertial>
+            <origin xyz="0 0 0.05" rpy="0 0 0"/>
+            <mass value="12" />
+            <inertia ixx="2.26" ixy="0.0" ixz="0.0" iyy="6.26" iyz="0.0" izz="8.5" />
+        </inertial>
 </link>
 <joint name="down_manipulator__rotation_base" type="revolute">
@@ -140,4 +212,15 @@
         <origin xyz="0 0 ${0.5*dmh}"/>
     </visual>
+    <collision>
+            <origin xyz="0 0 0.05" rpy="0 0 0"/>
+            <geometry>
+                <box size="2.5 1.5 0.1" />
+            </geometry>
+        </collision>
+        <inertial>
+            <origin xyz="0 0 0.05" rpy="0 0 0"/>
+            <mass value="12" />
+            <inertia ixx="2.26" ixy="0.0" ixz="0.0" iyy="6.26" iyz="0.0" izz="8.5" />
+        </inertial>
 </link>
 <joint name="down_manipulator__down_manipulator_joint" type="fixed">
@@ -154,4 +237,15 @@
         <origin rpy="1.57075 0 0" xyz="0 0 0"/>
     </visual>
+    <collision>
+            <origin xyz="0 0 0.05" rpy="0 0 0"/>
+            <geometry>
+                <box size="2.5 1.5 0.1" />
+            </geometry>
+        </collision>
+        <inertial>
+            <origin xyz="0 0 0.05" rpy="0 0 0"/>
+            <mass value="12" />
+            <inertia ixx="2.26" ixy="0.0" ixz="0.0" iyy="6.26" iyz="0.0" izz="8.5" />
+        </inertial>
 </link>
 <joint name="up_manipulator_joint__down_manipulator_joint" type="revolute">
@@ -170,4 +264,15 @@
         <origin rpy="0 0 0" xyz="0 0 ${0.5*umh}"/>
     </visual>
+    <collision>
+            <origin xyz="0 0 0.05" rpy="0 0 0"/>
+            <geometry>
+                <box size="2.5 1.5 0.1" />
+            </geometry>
+        </collision>
+        <inertial>
+            <origin xyz="0 0 0.05" rpy="0 0 0"/>
+            <mass value="12" />
+            <inertia ixx="2.26" ixy="0.0" ixz="0.0" iyy="6.26" iyz="0.0" izz="8.5" />
+        </inertial>
 </link>
 <joint name="up_manipulator__up_manipulator_joint" type="fixed">
@@ -184,4 +289,15 @@
         <origin rpy="1.57075 0 0" xyz="0 0 0"/>
     </visual>
+    <collision>
+            <origin xyz="0 0 0.05" rpy="0 0 0"/>
+            <geometry>
+                <box size="2.5 1.5 0.1" />
+            </geometry>
+        </collision>
+        <inertial>
+            <origin xyz="0 0 0.05" rpy="0 0 0"/>
+            <mass value="12" />
+            <inertia ixx="2.26" ixy="0.0" ixz="0.0" iyy="6.26" iyz="0.0" izz="8.5" />
+        </inertial>
 </link>
 <joint name="manipulator_hand_joint__up_manipulator_joint" type="revolute">
@@ -200,4 +316,15 @@
         <origin rpy="0 0 0" xyz="0 0 ${0.5*mhh}"/>
     </visual>
+    <collision>
+            <origin xyz="0 0 0.05" rpy="0 0 0"/>
+            <geometry>
+                <box size="2.5 1.5 0.1" />
+            </geometry>
+        </collision>
+        <inertial>
+            <origin xyz="0 0 0.05" rpy="0 0 0"/>
+            <mass value="12" />
+            <inertia ixx="2.26" ixy="0.0" ixz="0.0" iyy="6.26" iyz="0.0" izz="8.5" />
+        </inertial>
 </link>
 <joint name="manipulator_hand__manipulator_hand_joint" type="fixed">
@@ -214,4 +341,15 @@
         <origin xyz="0 0 0"/>
     </visual>
+    <collision>
+            <origin xyz="0 0 0.05" rpy="0 0 0"/>
+            <geometry>
+                <box size="2.5 1.5 0.1" />
+            </geometry>
+        </collision>
+        <inertial>
+            <origin xyz="0 0 0.05" rpy="0 0 0"/>
+            <mass value="12" />
+            <inertia ixx="2.26" ixy="0.0" ixz="0.0" iyy="6.26" iyz="0.0" izz="8.5" />
+        </inertial>
 </link>
 <joint name="camera_holder_manipulator_hand_joint" type="fixed">
@@ -228,4 +366,15 @@
         <origin xyz="0 0 ${chh}"/>
     </visual>
+    <collision>
+            <origin xyz="0 0 0.05" rpy="0 0 0"/>
+            <geometry>
+                <box size="2.5 1.5 0.1" />
+            </geometry>
+        </collision>
+        <inertial>
+            <origin xyz="0 0 0.05" rpy="0 0 0"/>
+            <mass value="12" />
+            <inertia ixx="2.26" ixy="0.0" ixz="0.0" iyy="6.26" iyz="0.0" izz="8.5" />
+        </inertial>
 </link>
 <joint name="camera_link_camera_holder_joint" type="fixed">
@@ -241,5 +390,15 @@
         <material name="white"/>
         <origin rpy="0 1.57075 0" xyz="0 0 0"/>
-    </visual>
+    </visual><collision>
+            <origin xyz="0 0 0.05" rpy="0 0 0"/>
+            <geometry>
+                <box size="2.5 1.5 0.1" />
+            </geometry>
+        </collision>
+        <inertial>
+            <origin xyz="0 0 0.05" rpy="0 0 0"/>
+            <mass value="12" />
+            <inertia ixx="2.26" ixy="0.0" ixz="0.0" iyy="6.26" iyz="0.0" izz="8.5" />
+        </inertial>
 </link>
 <link name="silver_box">
@@ -251,4 +410,15 @@
         <origin rpy="-1.54 0 0" xyz="0 0.03 -0.03"/>
     </visual>
+    <collision>
+            <origin xyz="0 0 0.05" rpy="0 0 0"/>
+            <geometry>
+                <box size="2.5 1.5 0.1" />
+            </geometry>
+        </collision>
+        <inertial>
+            <origin xyz="0 0 0.05" rpy="0 0 0"/>
+            <mass value="12" />
+            <inertia ixx="2.26" ixy="0.0" ixz="0.0" iyy="6.26" iyz="0.0" izz="8.5" />
+        </inertial>
 </link>
 <joint name="silver__manipulator_hand_joint" type="fixed">
@@ -271,4 +441,15 @@
         <origin rpy="0 0 0" xyz="${0.5*(tjh+gx)} 0 ${-0.5*(gg+gz)}"/>
     </visual>
+    <collision>
+            <origin xyz="0 0 0.05" rpy="0 0 0"/>
+            <geometry>
+                <box size="2.5 1.5 0.1" />
+            </geometry>
+        </collision>
+        <inertial>
+            <origin xyz="0 0 0.05" rpy="0 0 0"/>
+            <mass value="12" />
+            <inertia ixx="2.26" ixy="0.0" ixz="0.0" iyy="6.26" iyz="0.0" izz="8.5" />
+        </inertial>
 </link>
 <link name="right_gripper">
@@ -280,4 +461,15 @@
         <origin rpy="0 0 0" xyz="${0.5*(tjh+gx)} 0 ${0.5*(gg+gz)}"/>
     </visual>
+    <collision>
+            <origin xyz="0 0 0.05" rpy="0 0 0"/>
+            <geometry>
+                <box size="2.5 1.5 0.1" />
+            </geometry>
+        </collision>
+        <inertial>
+            <origin xyz="0 0 0.05" rpy="0 0 0"/>
+            <mass value="12" />
+            <inertia ixx="2.26" ixy="0.0" ixz="0.0" iyy="6.26" iyz="0.0" izz="8.5" />
+        </inertial>
 </link>
 <joint name="left_gripper__tool_joint" type="fixed">

Commit message: .

File: dobot_viz/urdf/dobot_viz.urdf.xacro (robot description, xacro)
@@ -66,10 +66,10 @@
             <origin xyz="0 0 0.05" rpy="0 0 0"/>
             <geometry>
-                <box size="2.5 1.5 0.1" />
-            </geometry>
-        </collision>
-        <inertial>
-            <origin xyz="0 0 0.05" rpy="0 0 0"/>
-            <mass value="12" />
+                <box size="0.01 0.01 0.01" />
+            </geometry>
+        </collision>
+        <inertial>
+            <origin xyz="0 0 0.05" rpy="0 0 0"/>
+            <mass value="0.001" />
             <inertia ixx="2.26" ixy="0.0" ixz="0.0" iyy="6.26" iyz="0.0" izz="8.5" />
         </inertial>
@@ -86,10 +86,10 @@
             <origin xyz="0 0 0.05" rpy="0 0 0"/>
             <geometry>
-                <box size="2.5 1.5 0.1" />
-            </geometry>
-        </collision>
-        <inertial>
-            <origin xyz="0 0 0.05" rpy="0 0 0"/>
-            <mass value="12" />
+                <box size="0.01 0.01 0.01" />
+            </geometry>
+        </collision>
+        <inertial>
+            <origin xyz="0 0 0.05" rpy="0 0 0"/>
+            <mass value="0.001" />
             <inertia ixx="2.26" ixy="0.0" ixz="0.0" iyy="6.26" iyz="0.0" izz="8.5" />
         </inertial>
@@ -111,10 +111,10 @@
             <origin xyz="0 0 0.05" rpy="0 0 0"/>
             <geometry>
-                <box size="2.5 1.5 0.1" />
-            </geometry>
-        </collision>
-        <inertial>
-            <origin xyz="0 0 0.05" rpy="0 0 0"/>
-            <mass value="12" />
+                <box size="0.01 0.01 0.01" />
+            </geometry>
+        </collision>
+        <inertial>
+            <origin xyz="0 0 0.05" rpy="0 0 0"/>
+            <mass value="0.001" />
             <inertia ixx="2.26" ixy="0.0" ixz="0.0" iyy="6.26" iyz="0.0" izz="8.5" />
         </inertial>
@@ -126,4 +126,5 @@
     <limit effort="1000.0" lower="-1.5708" upper="1.5708" velocity="0.5"/>
     <origin rpy="0 0 0" xyz="0 0 ${0.5*(bh+rbh)}"/>
+    <dynamics damping="100.0" friction="100.0"/>
 </joint>
 <link name="left_manipulator_handler">
@@ -138,10 +139,10 @@
             <origin xyz="0 0 0.05" rpy="0 0 0"/>
             <geometry>
-                <box size="2.5 1.5 0.1" />
-            </geometry>
-        </collision>
-        <inertial>
-            <origin xyz="0 0 0.05" rpy="0 0 0"/>
-            <mass value="12" />
+                <box size="0.01 0.01 0.01" />
+            </geometry>
+        </collision>
+        <inertial>
+            <origin xyz="0 0 0.05" rpy="0 0 0"/>
+            <mass value="0.001" />
             <inertia ixx="2.26" ixy="0.0" ixz="0.0" iyy="6.26" iyz="0.0" izz="8.5" />
         </inertial>
@@ -158,10 +159,10 @@
             <origin xyz="0 0 0.05" rpy="0 0 0"/>
             <geometry>
-                <box size="2.5 1.5 0.1" />
-            </geometry>
-        </collision>
-        <inertial>
-            <origin xyz="0 0 0.05" rpy="0 0 0"/>
-            <mass value="12" />
+                <box size="0.01 0.01 0.01" />
+            </geometry>
+        </collision>
+        <inertial>
+            <origin xyz="0 0 0.05" rpy="0 0 0"/>
+            <mass value="0.001" />
             <inertia ixx="2.26" ixy="0.0" ixz="0.0" iyy="6.26" iyz="0.0" izz="8.5" />
         </inertial>
@@ -171,4 +172,5 @@
     <child link="left_manipulator_handler"/>
     <origin xyz="0 0 0"/>
+    <dynamics damping="100.0" friction="100.0"/>
 </joint>
 <joint name="right_manipulator_handler__rotation_base" type="fixed">
@@ -176,4 +178,5 @@
     <child link="right_manipulator_handler"/>
     <origin xyz="0 0 0"/>
+    <dynamics damping="100.0" friction="100.0"/>
 </joint>
 <link name="down_manipulator_joint">
@@ -188,10 +191,10 @@
             <origin xyz="0 0 0.05" rpy="0 0 0"/>
             <geometry>
-                <box size="2.5 1.5 0.1" />
-            </geometry>
-        </collision>
-        <inertial>
-            <origin xyz="0 0 0.05" rpy="0 0 0"/>
-            <mass value="12" />
+                <box size="0.01 0.01 0.01" />
+            </geometry>
+        </collision>
+        <inertial>
+            <origin xyz="0 0 0.05" rpy="0 0 0"/>
+            <mass value="0.001" />
             <inertia ixx="2.26" ixy="0.0" ixz="0.0" iyy="6.26" iyz="0.0" izz="8.5" />
         </inertial>
@@ -203,4 +206,5 @@
     <child link="down_manipulator_joint"/>
     <origin xyz="0 0 ${wbh-bh}"/>
+    <dynamics damping="100.0" friction="100.0"/>
 </joint>
 <link name="down_manipulator">
@@ -215,10 +219,10 @@
             <origin xyz="0 0 0.05" rpy="0 0 0"/>
             <geometry>
-                <box size="2.5 1.5 0.1" />
-            </geometry>
-        </collision>
-        <inertial>
-            <origin xyz="0 0 0.05" rpy="0 0 0"/>
-            <mass value="12" />
+                <box size="0.01 0.01 0.01" />
+            </geometry>
+        </collision>
+        <inertial>
+            <origin xyz="0 0 0.05" rpy="0 0 0"/>
+            <mass value="0.001" />
             <inertia ixx="2.26" ixy="0.0" ixz="0.0" iyy="6.26" iyz="0.0" izz="8.5" />
         </inertial>
@@ -228,4 +232,5 @@
     <child link="down_manipulator"/>
     <origin xyz="0 0 0"/>
+    <dynamics damping="100.0" friction="100.0"/>
 </joint>
 <link name="up_manipulator_joint">
@@ -240,10 +245,10 @@
             <origin xyz="0 0 0.05" rpy="0 0 0"/>
             <geometry>
-                <box size="2.5 1.5 0.1" />
-            </geometry>
-        </collision>
-        <inertial>
-            <origin xyz="0 0 0.05" rpy="0 0 0"/>
-            <mass value="12" />
+                <box size="0.01 0.01 0.01" />
+            </geometry>
+        </collision>
+        <inertial>
+            <origin xyz="0 0 0.05" rpy="0 0 0"/>
+            <mass value="0.001" />
             <inertia ixx="2.26" ixy="0.0" ixz="0.0" iyy="6.26" iyz="0.0" izz="8.5" />
         </inertial>
@@ -255,4 +260,5 @@
     <limit effort="1000.0" lower="-1.5708" upper="1.5708" velocity="0.5"/>
     <origin rpy="0 ${pi/2} 0" xyz="0 0 ${dmh}"/>
+    <dynamics damping="100.0" friction="100.0"/>
 </joint>
 <link name="up_manipulator">
@@ -267,10 +273,10 @@
             <origin xyz="0 0 0.05" rpy="0 0 0"/>
             <geometry>
-                <box size="2.5 1.5 0.1" />
-            </geometry>
-        </collision>
-        <inertial>
-            <origin xyz="0 0 0.05" rpy="0 0 0"/>
-            <mass value="12" />
+                <box size="0.01 0.01 0.01" />
+            </geometry>
+        </collision>
+        <inertial>
+            <origin xyz="0 0 0.05" rpy="0 0 0"/>
+            <mass value="0.001" />
             <inertia ixx="2.26" ixy="0.0" ixz="0.0" iyy="6.26" iyz="0.0" izz="8.5" />
         </inertial>
@@ -280,4 +286,5 @@
     <child link="up_manipulator"/>
     <origin xyz="0 0 0"/>
+    <dynamics damping="100.0" friction="100.0"/>
 </joint>
 <link name="manipulator_hand_joint">
@@ -292,10 +299,10 @@
             <origin xyz="0 0 0.05" rpy="0 0 0"/>
             <geometry>
-                <box size="2.5 1.5 0.1" />
-            </geometry>
-        </collision>
-        <inertial>
-            <origin xyz="0 0 0.05" rpy="0 0 0"/>
-            <mass value="12" />
+                <box size="0.01 0.01 0.01" />
+            </geometry>
+        </collision>
+        <inertial>
+            <origin xyz="0 0 0.05" rpy="0 0 0"/>
+            <mass value="0.001" />
             <inertia ixx="2.26" ixy="0.0" ixz="0.0" iyy="6.26" iyz="0.0" izz="8.5" />
         </inertial>
@@ -307,4 +314,5 @@
     <limit effort="1000.0" lower="-1.5708" upper="1.5708" velocity="0.5"/>
     <origin rpy="0 0 0" xyz="0 0 ${umh}"/>
+    <dynamics damping="100.0" friction="100.0"/>
 </joint>
 <link name="manipulator_hand">
@@ -319,10 +327,10 @@
             <origin xyz="0 0 0.05" rpy="0 0 0"/>
             <geometry>
-                <box size="2.5 1.5 0.1" />
-            </geometry>
-        </collision>
-        <inertial>
-            <origin xyz="0 0 0.05" rpy="0 0 0"/>
-            <mass value="12" />
+                <box size="0.01 0.01 0.01" />
+            </geometry>
+        </collision>
+        <inertial>
+            <origin xyz="0 0 0.05" rpy="0 0 0"/>
+            <mass value="0.001" />
             <inertia ixx="2.26" ixy="0.0" ixz="0.0" iyy="6.26" iyz="0.0" izz="8.5" />
         </inertial>
@@ -332,4 +340,5 @@
     <child link="manipulator_hand"/>
     <origin xyz="0 0 0"/>
+    <dynamics damping="100.0" friction="100.0"/>
 </joint>
 <link name="camera_holder">
@@ -344,10 +353,10 @@
             <origin xyz="0 0 0.05" rpy="0 0 0"/>
             <geometry>
-                <box size="2.5 1.5 0.1" />
-            </geometry>
-        </collision>
-        <inertial>
-            <origin xyz="0 0 0.05" rpy="0 0 0"/>
-            <mass value="12" />
+                <box size="0.01 0.01 0.01" />
+            </geometry>
+        </collision>
+        <inertial>
+            <origin xyz="0 0 0.05" rpy="0 0 0"/>
+            <mass value="0.001" />
             <inertia ixx="2.26" ixy="0.0" ixz="0.0" iyy="6.26" iyz="0.0" izz="8.5" />
         </inertial>
@@ -357,4 +366,5 @@
     <child link="camera_holder"/>
     <origin xyz="0 0 ${mhh+0.5*chh}"/>
+    <dynamics damping="100.0" friction="100.0"/>
 </joint>
 <link name="camera_link">
@@ -369,10 +379,10 @@
             <origin xyz="0 0 0.05" rpy="0 0 0"/>
             <geometry>
-                <box size="2.5 1.5 0.1" />
-            </geometry>
-        </collision>
-        <inertial>
-            <origin xyz="0 0 0.05" rpy="0 0 0"/>
-            <mass value="12" />
+                <box size="0.01 0.01 0.01" />
+            </geometry>
+        </collision>
+        <inertial>
+            <origin xyz="0 0 0.05" rpy="0 0 0"/>
+            <mass value="0.001" />
             <inertia ixx="2.26" ixy="0.0" ixz="0.0" iyy="6.26" iyz="0.0" izz="8.5" />
         </inertial>
@@ -382,4 +392,5 @@
     <child link="camera_link"/>
     <origin xyz="0 0 0"/>
+    <dynamics damping="100.0" friction="100.0"/>
 </joint>
 <link name="tool_joint">
@@ -393,10 +404,10 @@
             <origin xyz="0 0 0.05" rpy="0 0 0"/>
             <geometry>
-                <box size="2.5 1.5 0.1" />
-            </geometry>
-        </collision>
-        <inertial>
-            <origin xyz="0 0 0.05" rpy="0 0 0"/>
-            <mass value="12" />
+                <box size="0.01 0.01 0.01" />
+            </geometry>
+        </collision>
+        <inertial>
+            <origin xyz="0 0 0.05" rpy="0 0 0"/>
+            <mass value="0.001" />
             <inertia ixx="2.26" ixy="0.0" ixz="0.0" iyy="6.26" iyz="0.0" izz="8.5" />
         </inertial>
@@ -413,10 +424,10 @@
             <origin xyz="0 0 0.05" rpy="0 0 0"/>
             <geometry>
-                <box size="2.5 1.5 0.1" />
-            </geometry>
-        </collision>
-        <inertial>
-            <origin xyz="0 0 0.05" rpy="0 0 0"/>
-            <mass value="12" />
+                <box size="0.01 0.01 0.01" />
+            </geometry>
+        </collision>
+        <inertial>
+            <origin xyz="0 0 0.05" rpy="0 0 0"/>
+            <mass value="0.001" />
             <inertia ixx="2.26" ixy="0.0" ixz="0.0" iyy="6.26" iyz="0.0" izz="8.5" />
         </inertial>
@@ -426,4 +437,5 @@
     <child link="silver_box"/>
     <origin xyz="0 0 0"/>
+    <dynamics damping="100.0" friction="100.0"/>
 </joint>
 <joint name="tool_joint__manipulator_hand_joint" type="continuous">
@@ -432,4 +444,5 @@
     <axis xyz="1 0 0"/>
     <origin xyz="${0.5*(mhx+tjh)} 0 ${mhh-0.5*mhy}" rpy="1.57 0 0"/>
+    <dynamics damping="100.0" friction="100.0"/>
 </joint>
 <link name="left_gripper">
@@ -444,10 +457,10 @@
             <origin xyz="0 0 0.05" rpy="0 0 0"/>
             <geometry>
-                <box size="2.5 1.5 0.1" />
-            </geometry>
-        </collision>
-        <inertial>
-            <origin xyz="0 0 0.05" rpy="0 0 0"/>
-            <mass value="12" />
+                <box size="0.01 0.01 0.01" />
+            </geometry>
+        </collision>
+        <inertial>
+            <origin xyz="0 0 0.05" rpy="0 0 0"/>
+            <mass value="0.001" />
             <inertia ixx="2.26" ixy="0.0" ixz="0.0" iyy="6.26" iyz="0.0" izz="8.5" />
         </inertial>
@@ -464,10 +477,10 @@
             <origin xyz="0 0 0.05" rpy="0 0 0"/>
             <geometry>
-                <box size="2.5 1.5 0.1" />
-            </geometry>
-        </collision>
-        <inertial>
-            <origin xyz="0 0 0.05" rpy="0 0 0"/>
-            <mass value="12" />
+                <box size="0.01 0.01 0.01" />
+            </geometry>
+        </collision>
+        <inertial>
+            <origin xyz="0 0 0.05" rpy="0 0 0"/>
+            <mass value="0.001" />
             <inertia ixx="2.26" ixy="0.0" ixz="0.0" iyy="6.26" iyz="0.0" izz="8.5" />
         </inertial>
@@ -477,4 +490,5 @@
     <child link="left_gripper"/>
     <origin xyz="0 0 0"/>
+    <dynamics damping="100.0" friction="100.0"/>
 </joint>
 <joint name="right_gripper__tool_joint" type="fixed">
@@ -482,4 +496,6 @@
     <child link="right_gripper"/>
     <origin xyz="0 0 0"/>
-</joint>
+    <dynamics damping="100.0" friction="100.0"/>
+</joint>
+<xacro:include filename="dobot_gazebo.xacro" />
 </robot>
