Commit message: .

File: dobot_viz/urdf/dobot_gazebo.xacro (robot description, xacro)
@@ -27,4 +27,5 @@
             <joint_name>manipulator_hand_joint__up_manipulator_joint</joint_name>
             <joint_name>tool_joint__manipulator_hand_joint</joint_name>
+            <joint_name>rover_world_joint</joint_name>
         </plugin>
     </gazebo>

File: dobot_viz/urdf/dobot_viz.urdf.xacro (robot description, xacro)
@@ -51,4 +51,28 @@
 </material>
 <link name="world"></link>
+<joint name="rover_world_joint" type="floating">
+    <origin xyz="2.5 0.0 0" rpy="0 0 0"/>
+    <parent link="base_link"/>
+    <child link="rover_body"/>
+</joint>
+<link name="rover_body">
+    <visual>
+        <geometry>
+            <box size="0.1 0.1 0.1"/>
+        </geometry>
+        <material name="white"/>
+    </visual>
+    <collision>
+            <origin xyz="0 0 0.05" rpy="0 0 0"/>
+            <geometry>
+                <box size="0.01 0.01 0.01" />
+            </geometry>
+        </collision>
+        <inertial>
+            <origin xyz="0 0 0.05" rpy="0 0 0"/>
+            <mass value="0.001" />
+            <inertia ixx="2.26" ixy="0.0" ixz="0.0" iyy="6.26" iyz="0.0" izz="8.5" />
+        </inertial>
+</link>
 <joint name="base_joint" type="fixed">
     <origin xyz="0.0 0.0 0" rpy="0 0 0"/>

Commit message: final working

File: dobot_viz/urdf/dobot_gazebo.xacro (robot description, xacro)
@@ -27,5 +27,4 @@
             <joint_name>manipulator_hand_joint__up_manipulator_joint</joint_name>
             <joint_name>tool_joint__manipulator_hand_joint</joint_name>
-            <joint_name>rover_world_joint</joint_name>
         </plugin>
     </gazebo>

File: dobot_viz/urdf/dobot_viz.urdf.xacro (robot description, xacro)
@@ -51,28 +51,4 @@
 </material>
 <link name="world"></link>
-<joint name="rover_world_joint" type="floating">
-    <origin xyz="2.5 0.0 0" rpy="0 0 0"/>
-    <parent link="base_link"/>
-    <child link="rover_body"/>
-</joint>
-<link name="rover_body">
-    <visual>
-        <geometry>
-            <box size="0.1 0.1 0.1"/>
-        </geometry>
-        <material name="white"/>
-    </visual>
-    <collision>
-            <origin xyz="0 0 0.05" rpy="0 0 0"/>
-            <geometry>
-                <box size="0.01 0.01 0.01" />
-            </geometry>
-        </collision>
-        <inertial>
-            <origin xyz="0 0 0.05" rpy="0 0 0"/>
-            <mass value="0.001" />
-            <inertia ixx="2.26" ixy="0.0" ixz="0.0" iyy="6.26" iyz="0.0" izz="8.5" />
-        </inertial>
-</link>
 <joint name="base_joint" type="fixed">
     <origin xyz="0.0 0.0 0" rpy="0 0 0"/>
@@ -522,4 +498,4 @@
     <dynamics damping="100.0" friction="100.0"/>
 </joint>
-<xacro:include filename="dobot_gazebo.xacro" />
+<!-- <xacro:include filename="dobot_gazebo.xacro" /> -->
 </robot>
